File: PCB/eagle/SmartSensorWifi.brd (EAGLE design)
At the start: 100 x 80 mm, 8 parts, among them IC1 AT45DB-S

Commit message: Updated board
Parts:
- added PH1: D1160_12, photo-elements:D11XX
- added R2: (no value), adafruit:0805-THM
Connections:
- new net N$13: U$2.P$14, WIFI1.40
- new net N$14: U$2.P$15, WIFI1.42
- new net N$15: PH1.2, R2.2, U$2.P$30
- net GND: now also R2.1
- net VCC: now also PH1.1, WIFI1.34
Routing:
- net GND: track 95.3 -> 227.7 mm, vias 6 -> 8
- net N$14: track 0.00 -> 129.1 mm, vias 0 -> 4
- net N$13: track 0.00 -> 125.3 mm, vias 0 -> 4
- net VCC: track 59.7 -> 157.5 mm, vias 1 -> 5
- net N$15: track 0.00 -> 63.0 mm, vias 0 -> 2
- net N$9: track 86.6 -> 98.9 mm
