File: PCB/eagle/SmartSensorWifi.sch (EAGLE design)
At the start: 8 parts, among them IC1 AT45DB-S

Commit message: Updated board
Parts:
- added PH1: D1160_12, photo-elements:D1160_12
- added R2: (no value), adafruit:FLIPFLOP-RES
Connections:
- new net N$13: U$2.RX, WIFI1.UART0_TX
- new net N$14: U$2.TX, WIFI1.UART0_RX
- new net N$15: PH1.2, R2.2, U$2.A1
- net GND: now also R2.1
- net VCC: now also PH1.1, WIFI1.VDDIO
Changed lines of the file:
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@@
 <part name="SUPPLY9" library="supply2" deviceset="GND" device=""/>
 <part name="SUPPLY10" library="supply2" deviceset="GND" device=""/>
+<part name="SUPPLY11" library="supply2" deviceset="VCC" device=""/>
+<part name="PH1" library="photo-elements" deviceset="D11" device="" technology="60_12"/>
+<part name="R2" library="adafruit" deviceset="FLIPFLOP-RES" device=""/>
+<part name="SUPPLY12" library="supply2" deviceset="GND" device=""/>
+<part name="SUPPLY13" library="supply2" deviceset="VCC" device=""/>
 </parts>
 <sheets>
@@
 <instance part="SUPPLY9" gate="GND" x="-5.08" y="-20.32" rot="R90"/>
 <instance part="SUPPLY10" gate="GND" x="-5.08" y="15.24" rot="R90"/>
+<instance part="SUPPLY11" gate="G$1" x="-5.08" y="-12.7" rot="R270"/>
+<instance part="PH1" gate="G$1" x="-10.16" y="48.26" rot="MR270"/>
+<instance part="R2" gate="G$1" x="5.08" y="48.26" rot="MR0"/>
+<instance part="SUPPLY12" gate="GND" x="12.7" y="48.26" rot="MR270"/>
+<instance part="SUPPLY13" gate="G$1" x="-17.78" y="48.26" rot="MR270"/>
 </instances>
 <busses>
@@
 <pinref part="WIFI1" gate="G$1" pin="GND4"/>
 <pinref part="SUPPLY10" gate="GND" pin="GND"/>
+</segment>
+<segment>
+<pinref part="R2" gate="G$1" pin="1"/>
+<pinref part="SUPPLY12" gate="GND" pin="GND"/>
 </segment>
 </net>
@@
 <junction x="10.16" y="-7.62"/>
 </segment>
+<segment>
+<pinref part="WIFI1" gate="G$1" pin="VDDIO"/>
+<pinref part="SUPPLY11" gate="G$1" pin="VCC"/>
+</segment>
+<segment>
+<pinref part="PH1" gate="G$1" pin="1"/>
+<pinref part="SUPPLY13" gate="G$1" pin="VCC"/>
+</segment>
 </net>
 <net name="N$2" class="0">
@@
 <wire x1="104.14" y1="-17.78" x2="104.14" y2="-12.7" width="0.1524" layer="91"/>
 <wire x1="104.14" y1="-12.7" x2="63.5" y2="-12.7" width="0.1524" layer="91"/>
-<wire x1="63.5" y1="-12.7" x2="63.5" y2="-43.18" width="0.1524" layer="91"/>
-<wire x1="63.5" y1="-43.18" x2="12.7" y2="-43.18" width="0.1524" layer="91"/>
-<wire x1="12.7" y1="-43.18" x2="12.7" y2="-17.78" width="0.1524" layer="91"/>
+<wire x1="63.5" y1="-12.7" x2="63.5" y2="-33.02" width="0.1524" layer="91"/>
+<wire x1="63.5" y1="-33.02" x2="12.7" y2="-33.02" width="0.1524" layer="91"/>
+<wire x1="12.7" y1="-33.02" x2="12.7" y2="-17.78" width="0.1524" layer="91"/>
 <pinref part="U$2" gate="G$1" pin="MISO"/>
 <wire x1="12.7" y1="-17.78" x2="20.32" y2="-17.78" width="0.1524" layer="91"/>
@@
 <wire x1="0" y1="-17.78" x2="0" y2="17.78" width="0.1524" layer="91"/>
 <wire x1="0" y1="17.78" x2="12.7" y2="17.78" width="0.1524" layer="91"/>
+<junction x="12.7" y="17.78"/>
+<junction x="68.58" y="-27.94"/>
+<junction x="104.14" y="-25.4"/>
 </segment>
 </net>
@@
 </segment>
 </net>
+<net name="N$13" class="0">
+<segment>
+<pinref part="U$2" gate="G$1" pin="RX"/>
+<wire x1="45.72" y1="-12.7" x2="50.8" y2="-12.7" width="0.1524" layer="91"/>
+<wire x1="50.8" y1="-12.7" x2="50.8" y2="-27.94" width="0.1524" layer="91"/>
+<wire x1="50.8" y1="-27.94" x2="2.54" y2="-27.94" width="0.1524" layer="91"/>
+<pinref part="WIFI1" gate="G$1" pin="UART0_TX"/>
+<wire x1="2.54" y1="-27.94" x2="2.54" y2="-5.08" width="0.1524" layer="91"/>
+<wire x1="2.54" y1="-5.08" x2="-7.62" y2="-5.08" width="0.1524" layer="91"/>
+</segment>
+</net>
+<net name="N$14" class="0">
+<segment>
+<pinref part="U$2" gate="G$1" pin="TX"/>
+<wire x1="45.72" y1="-15.24" x2="48.26" y2="-15.24" width="0.1524" layer="91"/>
+<wire x1="48.26" y1="-15.24" x2="48.26" y2="-25.4" width="0.1524" layer="91"/>
+<wire x1="48.26" y1="-25.4" x2="5.08" y2="-25.4" width="0.1524" layer="91"/>
+<pinref part="WIFI1" gate="G$1" pin="UART0_RX"/>
+<wire x1="5.08" y1="-25.4" x2="5.08" y2="0" width="0.1524" layer="91"/>
+<wire x1="5.08" y1="0" x2="-7.62" y2="0" width="0.1524" layer="91"/>
+</segment>
+</net>
+<net name="N$15" class="0">
+<segment>
+<pinref part="PH1" gate="G$1" pin="2"/>
+<pinref part="R2" gate="G$1" pin="2"/>
+<wire x1="-5.08" y1="48.26" x2="-2.54" y2="48.26" width="0.1524" layer="91"/>
+<pinref part="U$2" gate="G$1" pin="A1"/>
+<wire x1="-2.54" y1="48.26" x2="0" y2="48.26" width="0.1524" layer="91"/>
+<wire x1="20.32" y1="10.16" x2="7.62" y2="10.16" width="0.1524" layer="91"/>
+<wire x1="7.62" y1="10.16" x2="7.62" y2="45.72" width="0.1524" layer="91"/>
+<wire x1="7.62" y1="45.72" x2="-2.54" y2="45.72" width="0.1524" layer="91"/>
+<wire x1="-2.54" y1="45.72" x2="-2.54" y2="48.26" width="0.1524" layer="91"/>
+</segment>
+</net>
