File: PCB/SmartSensorWifi/RaspberryShield.brd (EAGLE design)
At the start: 100 x 80 mm, 4 parts

Commit message: Updated the PCB/BRD files
Parts:
- added TMP36: (no value), SparkFun-Sensors:TO-92
- renumbered PH1 to PR1, X1 to ADC1
Connections:
- new net A0: ADC1.P$1, PR1.1, R1.2
- net 3V3: now also ADC1.P$16, R1.1, TMP36.1
- net 5V: no longer ADC1.P$16, R1.1
- net A1: now also ADC1.P$2, TMP36.2; no longer ADC1.P$1, PR1.1, R1.2
- net GND: now also TMP36.3
Routing:
- net 5V: track 47.3 -> 0.00 mm, vias 2 -> 0
- net GND: track 75.3 -> 110.2 mm, vias 2 -> 3
- net N$10: track 0.00 -> 27.0 mm, vias 0 -> 1
- net 3V3: track 43.6 -> 68.9 mm, vias 0 -> 1
- net N$9: track 0.00 -> 23.8 mm, vias 0 -> 1
- net N$8: track 0.00 -> 19.6 mm, vias 0 -> 1
- net A0: track 0.00 -> 18.1 mm
- net N$11: track 0.00 -> 14.7 mm, vias 0 -> 1
- net N$12: track 0.00 -> 9.46 mm, vias 0 -> 1
- net N$1: track 0.00 -> 4.83 mm, vias 0 -> 1
- net A1: track 18.1 -> 19.8 mm
