File: PCB/SmartSensorWifi/RaspberryShield.sch (EAGLE design)
At the start: 4 parts

Commit message: Updated the PCB/BRD files
Parts:
- added TMP36: (no value), SparkFun-Sensors:TMP36GT9
- renumbered PH1 to PR1, X1 to ADC1
Connections:
- new net A0: ADC1.CH0, PR1.1, R1.2
- net 3V3: now also ADC1.VDD, R1.1, TMP36.VCC
- net 5V: no longer ADC1.VDD, R1.1
- net A1: now also ADC1.CH1, TMP36.VOUT; no longer ADC1.CH0, PR1.1, R1.2
- net GND: now also TMP36.GND
