File: PCB/SmartSensorWifi/SmartSensorWifi.brd (EAGLE design)
At the start: 100 x 80 mm, 8 parts, among them IC1 AT45DB-S

Commit message: Updated the eagle files
Parts:
- removed Q1: (no value), special:Q
- removed R1: (no value), adafruit:0805-THM
- removed S1: SPST, adafruit:JUDCOSPST
- removed WIFI1: WIZFI210, SmartSensorWifi:WIZFI210
- added CN1: (no value), adafruit:JST-PH-2-THM
- added PH1: D1160_12, photo-elements:D11XX
- added Q2: (no value), adafruit:TC38H
- added R2: 220, adafruit:0207/12
- added R3: (no value), adafruit:0207/12
- added U$4: WIZFISTACKED, SmartSensorWifi:WIZFI210STACKABLE
- moved IC1 66.3 mm to (63.5, 10.2), turned to 0 degrees
- moved U$1 55.5 mm to (81.3, 52.1), turned to 90 degrees
- moved U$3 25.0 mm to (87.6, 72.4), turned to 0 degrees
- moved U$2 18.0 mm to (62.2, 43.2), turned to 270 degrees
Connections:
- removed net N$11: IC1.4, U$2.P$7
- removed net N$12: R1.2, S1.T, U$2.P$8
- removed net N$6: IC1.8, U$2.P$19
- removed net N$7: IC1.2, U$2.P$18
- removed net N$8: IC1.1, U$2.P$17
- removed net N$9: IC1.3, IC1.5, IC1.6, U$2.P$33, WIFI1.32
- removed net VCC: S1.P, U$1.1, U$2.P$23
- new net 3V3: IC1.3, U$2.P$33, U$4.VIN3V3
- new net 5V: R2.1, R3.1, U$1.1, U$2.P$23, U$4.VDDIO
- new net A1: PH1.1, R2.2, U$2.P$30
- new net CS_FLASH: IC1.4, U$2.P$8
- new net CS_WIFI: U$2.P$7, U$4.SPI_CS
- new net GND2: U$4.GND2
- new net GND3: U$4.GND3
- new net GND4: U$4.GND4
- new net MISO: IC1.8, U$2.P$19, U$4.SPI_MISO
- new net MOSI: IC1.1, U$2.P$17, U$4.SPI_MOSI
- new net PSHBTN: CN1.2, R3.2, U$2.P$10
- new net S$1: PH1.2, U$4.GND
- new net SCK: IC1.2, U$2.P$18, U$4.SPI_CLK
- new net WIFI_HOSTWAKEUP: U$2.P$9, U$4.GPIO19
- net GND: now also CN1.1; no longer R1.1, U$2.P$12, WIFI1.1, WIFI1.18, WIFI1.31, WIFI1.48
- net N$10: no longer U$3.+2
- net N$2: now also Q2.2; no longer Q1.1
- net N$3: now also Q2.1; no longer Q1.2
- net VBAT: now also U$4.VBAT; no longer WIFI1.9
- net VOUT_1V8: now also U$4.VOUT_1V8; no longer WIFI1.17
Routing:
- net 5V: track 0.00 -> 124.3 mm, vias 0 -> 6
- net MOSI: track 0.00 -> 123.9 mm, vias 0 -> 2
- net CS_WIFI: track 0.00 -> 108.9 mm
- net S$1: track 0.00 -> 91.5 mm
- net N$9: track 86.6 -> 0.00 mm, vias 2 -> 0
- net 3V3: track 0.00 -> 84.5 mm, vias 0 -> 2
- net SCK: track 0.00 -> 75.9 mm
- net WIFI_HOSTWAKEUP: track 0.00 -> 75.0 mm
- net MISO: track 0.00 -> 68.5 mm
- net VCC: track 59.7 -> 0.00 mm, vias 1 -> 0
- net N$11: track 57.5 -> 0.00 mm, vias 2 -> 0
- net CS_FLASH: track 0.00 -> 56.4 mm, vias 0 -> 2
- net N$3: track 67.6 -> 12.7 mm
- net N$2: track 59.3 -> 8.15 mm
- net N$10: track 76.7 -> 27.9 mm, vias 2 -> 0
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Other:
- board size 100 x 80 mm -> 100 x 82.5 mm

Commit message: Updated the PCB/BRD files
Parts:
- moved U$4 115.1 mm to (83.3, 31.2), flipped to the bottom
- moved R3 7.98 mm to (86.1, 43.2), turned to 0 degrees
- moved U$3 0.25 mm to (87.9, 72.4)
Routing:
- net 3V3: track 84.5 -> 171.9 mm, vias 2 -> 1
- net MOSI: track 123.9 -> 55.6 mm
- net CS_WIFI: track 108.9 -> 50.2 mm
- net MISO: track 68.5 -> 30.6 mm
- net WIFI_HOSTWAKEUP: track 75.0 -> 37.0 mm, vias 0 -> 2
- net SCK: track 75.9 -> 49.2 mm, vias 0 -> 1
- net S$1: track 91.5 -> 101.1 mm, vias 0 -> 1
- net S$3: track 0.00 -> 9.40 mm
- net PSHBTN: track 33.4 -> 26.1 mm
- net GND: track 111.9 -> 104.6 mm, vias 2 -> 1
- net CS_FLASH: track 56.4 -> 62.1 mm, vias 2 -> 1
- net 5V: track 124.3 -> 122.6 mm, vias 6 -> 0
- net A1: track 30.3 -> 31.2 mm
